File: PCB_Tarjeta_DevOps/PCB_Tarjeta_DevOps.kicad_pcb (KiCad board)
At the start: 2 copper layers, 100 x 190 mm, 195 parts, among them J101 Conn_01x10_Pin, J102 Conn_01x10_Pin, J103 Conn_01x16_Pin, J104 Conn_01x16_Pin, J105 RJHSE-5384, J106 USB_C_Receptacle_USB2.0_16P, J401 Conn_01x02, J402 Conn_01x02, Q401 SS8050, SW101 SW_Push, SW102 SW_Push, SW103 SW_Push, SW104 SW_Push, SW105 SW_Push, SW106 SW_DPDT_x2, SW601 SW_Push, T701 H1102NL, U201 AZ1117CH2-3.3, U202 ST890CDR, U301 CH340G, U302 SRV05-4, U401 STM32F103CBTx, U501 DS1302Z+, U601 ITS4090QEPDXUMA1, U602 ITS4090QEPDXUMA1, U603 SRV05-4, U604 SRV05-4, U605 STM32F412ZGTx, U606 TLP290-4, U607 TLP290-4, U608 SRV05-4, U609 SRV05-4, U701 LAN8742A-CZ-TR, U702 SRV05-4, Y301 ASE-xxxMHz, Y401 ASE-xxxMHz, Y501 ASE-xxxMHz, Y601 ASE-xxxMHz, Y602 ASE-xxxMHz, Y701 ASE-xxxMHz

Commit message: Add files via upload
Other:
- board text added: "OCTOBER 2025"
- board text added: "PROTO_CONSOLE"
- board text added: "R.CASAS"
Changed lines of the file:
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@@
 		(layer "F.SilkS")
+	)
+	(gr_rect
+		(start 145.228 232.708)
+		(end 166.056 243.376)
+		(stroke
+			(width 0.25)
+			(type solid)
+		)
+		(fill no)
+		(layer "B.SilkS")
 	)
 	(gr_poly
@@
 		(layer "Edge.Cuts")
 	)
+	(gr_text "OCTOBER 2025"
+		(at 164.278 242.614 -0)
+		(layer "B.Cu")
+		(effects
+			(font
+				(size 1.5 1.5)
+				(thickness 0.25)
+				(bold yes)
+			)
+			(justify left bottom mirror)
+		)
+	)
+	(gr_text "PROTO_CONSOLE"
+		(at 164.659 235.756 0)
+		(layer "B.Cu")
+		(effects
+			(font
+				(size 1.5 1.5)
+				(thickness 0.25)
+				(bold yes)
+			)
+			(justify left bottom mirror)
+		)
+	)
+	(gr_text "R.CASAS"
+		(at 159.96 239.312 -0)
+		(layer "B.Cu")
+		(effects
+			(font
+				(size 1.5 1.5)
+				(thickness 0.25)
+				(bold yes)
+			)
+			(justify left bottom mirror)
+		)
+	)
 	(gr_text "FAULT"
